Commit message: Verified Fiducial SLAM

File: xxx_description/urdf/xxx_gazebo.xacro (robot description, xacro)
@@ -136,5 +136,5 @@
             <imageTopicName>image_raw</imageTopicName>
             <cameraInfoTopicName>camera_info</cameraInfoTopicName>
-            <frameName>camera</frameName>
+            <frameName>camera_optical</frameName>
             <hackBaseline>0.07</hackBaseline>
             <distortionK1>0.0</distortionK1>

File: xxx_description/urdf/xxx_sensor.xacro (robot description, xacro)
@@ -39,8 +39,14 @@
             </visual>
         </link>
+        <link name="camera_optical"/>
         <joint name="camera_joint" type="fixed">
             <parent link="base_link" />
             <child link="camera" />
             <origin xyz="0.317 0 0.1" rpy="0 0 0" />
+        </joint>
+        <joint name="camera_optical_joint" type="fixed">
+            <parent link="camera" />
+            <child link="camera_optical" />
+            <origin xyz="0 0 0" rpy="-1.570796325 0 -1.570796325" />
         </joint>
         <link name="ultrasonic1">
